File: hardware/kicad/OzSec2026-ESP32/OzSec2026-ESP32.kicad_sch (KiCad schematic)
At the start: 59 parts, among them J1 UART, J2 USB_C_Receptacle_USB2.0, J3 JTAG, J4 DISPLAY, J5 Conn_01x03_Socket, SW1 SW_Push, SW2 SW_Push, SW3 SW_Push, SW4 SW_Push, SW5 POWER, SW6 SW_Push, SW7 SW_Push, U1 USBLC6-2SC6, U2 ESP32-S3-WROOM-1, U3 TSOP38238, U4 ME4054BM5G-N, U5 TLV1117LV-33, X1 Simple_Addon_v2

Commit message: Update resistor value 1K -> 100R with updated LCSC part (C17408)
Co-Authored-By: Claude Sonnet 4.6 <noreply@anthropic.com>
Parts:
- R8: value 1K -> 100; LCSC C17513 -> C17408; Link https://www.lcsc.com/product-detail/C17513.html -> https://www.lcsc.com/product-detail/C17408.html
Changed lines of the file:
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@@
 			)
 		)
-		(property "Value" "1K"
+		(property "Value" "100"
 			(at 87.63 121.9199 0)
 			(effects
@@
 			)
 		)
-		(property "Link" "https://www.lcsc.com/product-detail/C17513.html"
+		(property "Link" "https://www.lcsc.com/product-detail/C17408.html"
 			(at 85.09 120.65 0)
 			(effects
@@
 			)
 		)
-		(property "LCSC" "C17513"
+		(property "LCSC" "C17408"
 			(at 85.09 120.65 0)
 			(effects
